File: WeMos-RFLink.sch (EAGLE design)
At the start: 11 parts, among them P1 PADSMALL

Commit message: V1.1 Transceiver on bottom shield + RGB LED
Parts:
- removed JP4: (no value), SparkFun-Connectors:M021X02_NO_SILK
- added C1: 100nF, _c2h:CAP0805-CAP
- added C2: 10uF, _c2h:CAP0805-CAP-LARGEPADS
- added D1: 1N4148, Seeed-Discrete:D-ESD-2P-CESD5V0D1
- added P2, P3: PADNORMAL, _c2h:PADNORMAL
- added WS2812: WS2812B, _c2h:WS2812BSMD
Connections:
- new net DO: P2.1, WS2812.DOUT
- new net VLED: C1.1, D1.2, WS2812.VDD
- net 3V3: now also C2.2, JP3.1, JP3.2; no longer JP4.1, JP4.2
- net 5V: now also D1.1
- net GND: now also C1.2, C2.1, P3.1, WS2812.GND; no longer JP3.1, JP3.2
- net GPIO0: now also WS2812.DIN
Other:
- moved on the sheet: JP3
